File: Neopixel_project_v3.0.kicad_sch (KiCad schematic)
At the start: 65 parts, among them J1 Conn_01x03_Pin, J3 Screw_Terminal_01x02, Q1 MMBT3904, Q2 MMBT3904, Q3 MMBT3904, Q4 MMBT3904, Q5 DO3407B, Q6 DO3407B, Q7 DO3407B, Q8 DO3407B, SW1 TS-1088-AR02016, SW2 TS-1088-AR02016, U1 ESP8685H4, U2 AL8843, U3 TD1469, U4 USBLC6-4SC6, Y1 Crystal_GND24

Commit message: silkscreen removed and layout printed
Other:
- company: (none) -> Scrarf
Changed lines of the file:
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@@
 		(date "2025-09-10")
 		(rev "3.0")
+		(company "Scrarf")
 	)
 	(junction
